File: schemas/spc-player/spc-player.sch (KiCad schematic (older format))
At the start: 3 parts

Commit message: update
Parts:
- gave numbers to parts that had none: 3
Changed lines of the file:
@@
 $EndDescr
 $Comp
-L snes-apu-connector:SNES_APU_CONN J?
+L snes-apu-connector:SNES_APU_CONN J1
 U 1 1 5E700C9A
 P 4400 2350
-F 0 "J?" H 4275 3165 50  0000 C CNN
+F 0 "J1" H 4275 3165 50  0000 C CNN
 F 1 "SNES_APU_CONN" H 4275 3074 50  0000 C CNN
 F 2 "" H 4400 2350 50  0001 C CNN
@@
 	3050 2600 3050 3050
 $Comp
-L MCU_Module:Arduino_UNO_R2 A?
+L MCU_Module:Arduino_UNO_R2 A1
 U 1 1 5E6EA817
 P 2250 2300
-F 0 "A?" H 2250 3481 50  0000 C CNN
+F 0 "A1" H 2250 3481 50  0000 C CNN
 F 1 "Arduino_UNO_R2" H 2250 3390 50  0000 C CNN
 F 2 "Module:Arduino_UNO_R2" H 2250 2300 50  0001 C CIN
@@
 	5550 1850 5550 3500
 $Comp
-L Connector:AudioJack2_Ground J?
+L Connector:AudioJack2_Ground J2
 U 1 1 5E716921
 P 5550 1650
-F 0 "J?" H 5370 1668 50  0000 R CNN
+F 0 "J2" H 5370 1668 50  0000 R CNN
 F 1 "AudioJack2_Ground" H 5370 1577 50  0000 R CNN
 F 2 "" H 5550 1650 50  0001 C CNN

Commit message: schema update
Parts:
- A1: value Arduino_UNO_R2 -> Arduino_Micro_R2; symbol MCU_Module:Arduino_UNO_R2 -> spc-player-rescue:Arduino_UNO_R2-MCU_Module
- J2: symbol Connector:AudioJack2_Ground -> spc-player-rescue:AudioJack2_Ground-Connector
Changed lines of the file:
@@
 	3050 2600 3050 3050
 $Comp
-L MCU_Module:Arduino_UNO_R2 A1
+L spc-player-rescue:Arduino_UNO_R2-MCU_Module A1
 U 1 1 5E6EA817
 P 2250 2300
 F 0 "A1" H 2250 3481 50  0000 C CNN
-F 1 "Arduino_UNO_R2" H 2250 3390 50  0000 C CNN
+F 1 "Arduino_Micro_R2" H 2250 3390 50  0000 C CNN
 F 2 "Module:Arduino_UNO_R2" H 2250 2300 50  0001 C CIN
 F 3 "https://www.arduino.cc/en/Main/arduinoBoardUno" H 2250 2300 50  0001 C CNN
@@
 	5550 1850 5550 3500
 $Comp
-L Connector:AudioJack2_Ground J2
+L spc-player-rescue:AudioJack2_Ground-Connector J2
 U 1 1 5E716921
 P 5550 1650
